File: hardware/V1.3/step-down.kicad_pcb (KiCad board)
At the start: 2 copper layers, 40 x 40 mm, 38 parts, among them J1 STACK-UP-HIGH, J2 STACK-UP-HIGH, P1 Black, P2 Green, Q1 FDS8449, U1 ZXCT1086, U2 AOZ1212, U3 DRILL, U4 DRILL, U5 DRILL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

Commit message: update pcb
Parts:
- U3, U4, U5, U6: footprint DRILL_NP -> kicad-libraries:DRILL_NP
Other:
- board text added: "Step Down Power Supply 1.3"
- board text removed: "Power Supply Step Down 1.3"

Commit message: change components to new standard components, oder version
Parts:
- C2, C3, C4, C5, C6, R6, R7, R8: footprint 0603E -> C0603E
- FB1, R4: footprint kicad-libraries:1206 -> R1206
- Fiducial_Mark (x2): footprint Fiducial_Mark -> kicad-libraries:Fiducial_Mark
- R1, R2, R3, R5: footprint 0603E -> R0603E
- U3, U4, U5, U6: footprint kicad-libraries:DRILL_NP -> DRILL_NP
- VAL: footprint CE_5mm -> kicad-libraries:CE_5mm
- VAL: footprint WEEE_7mm -> kicad-libraries:WEEE_7mm
- turned FB1 to 90 degrees
- turned VAL to 180 degrees
Connections:
- FB1 pad 1: AGND -> GND
- FB1 pad 2: GND -> AGND

Commit message: Add 3d information (tbc)
Parts:
- C1, C7: footprint ELKO_83 -> kicad-libraries:ELKO_83
- C2, C3, C4, C5, C6, R6, R7, R8: footprint C0603E -> kicad-libraries:C0603E
- D1: footprint SOD-123 -> kicad-libraries:SOD-123
- D2, D3, D4, D5: footprint SOD-128 -> kicad-libraries:SOD-128
- FB1, R4: footprint R1206 -> kicad-libraries:R1206
- J1, J2: footprint BTB08-ACS-TOP -> kicad-libraries:BTB08-ACS-TOP
- L1: footprint SRP7030 -> kicad-libraries:SRP7030
- P1, P2: footprint OQ_2P -> kicad-libraries:OQ_2P
- Q1: footprint SOIC-8-MOSFET -> kicad-libraries:SOIC-8-MOSFET
- R1, R2, R3, R5: footprint R0603E -> kicad-libraries:R0603E
- U1: footprint SOT23-5 -> kicad-libraries:SOT23-5
- U2: footprint SO-8 -> kicad-libraries:SO-8
- U3, U4, U5, U6: footprint DRILL_NP -> kicad-libraries:DRILL_NP
